File: breakout.kicad_pcb (KiCad board)
At the start: 2 copper layers, 51.2 x 61 mm, 9 parts, among them J1 Conn_01x32, J2 Conn_02x16_Top_Bottom, U1 74ALVC164245, U2 74ALVC164245

Commit message: sad
Routing:
- net /DATA_DIR: track 39.0 -> 41.1 mm
Changed lines of the file:
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@@
 	)
 	(segment
-		(start 157.526 70.446)
-		(end 157.526 102.14766)
+		(start 158.6 103.2)
+		(end 156.9 104.9)
+		(width 0.2)
+		(layer "F.Cu")
+		(net 65)
+	)
+	(segment
+		(start 156.9 104.9)
+		(end 154.25 104.9)
 		(width 0.2)
 		(layer "F.Cu")
@@
 	(segment
 		(start 155.48 68.4)
-		(end 157.526 70.446)
+		(end 158.6 71.52)
 		(width 0.2)
 		(layer "F.Cu")
@@
 	)
 	(segment
-		(start 157.526 102.14766)
-		(end 154.77366 104.9)
+		(start 158.6 71.52)
+		(end 158.6 103.2)
 		(width 0.2)
 		(layer "F.Cu")
-		(net 65)
-	)
-	(segment
-		(start 154.77366 104.9)
-		(end 154.25 104.9)
-		(width 0.2)
-		(layer "F.Cu")
